File: hardware/kicad/Eurocard-HV-piezo-driver.kicad_pcb (KiCad board)
At the start: 4 copper layers, 160 x 100 mm, 171 parts, among them J1 VG64C, J2 2X8_LOW_PROFILE_JUMPER, J3 2X4_LOW_PROFILE_JUMPER, J4 2X8_LOW_PROFILE_JUMPER, J5 1x7 2.00mm, SW2 SWITCH-TACTILE, T1 ATB3225, U1 DRV2700, U2 MIC5209, U3 LM7171, U4 LM7171, U6 OPA2172, U7 AD8421, U8 74AHCT1G02, U9 MK20DX256VLH7, X1 UMC, X2 16MHz 7.2pF

Commit message: Add board QR code and source link to ion-optics repository
Point the printed source URL and a new silkscreen-only QR footprint to
https://github.com/dyknapp/-ion-optics-hv. Preserve JQI attribution and
record the published Documentation Location in the signed project docs.

Use Q error correction, 0.45 mm modules and a four-module quiet border
in an 18.45 mm square below the exposed RF-shield rim. Keep the artwork
board-only and excluded from BOM/placement files; add its local library.

Validation: decode the mask-subtracted silkscreen plot at three sizes to
the exact URL. All existing electrical geometry/footprints are unchanged.
DRC remains 557, schematic parity 137 and unconnected items zero, with
no findings involving the QR code or updated source label.
Parts:
- added QR1: https://github.com/dyknapp/-ion-optics-hv, IonOptics:QR_Documentation, F.Cu at (151.2, 143.8)
Other:
- board text added: "Source: github.com/dyknapp/-ion-optics-hv"
- board text removed: "Upstream: github.com/JQIamo/hv-piezo-driver"
